File: hardware/hybrid-panda/HybridPanda.kicad_pcb (KiCad board)
At the start: 4 copper layers, 50.9 x 46.7 mm, 125 parts, among them J1 SWD, P1 TYPE-C-31-M-04, Q1 DDTA143ECA-7-F P08, Q2 DDTA143ECA-7-F P08, Q3 PDTC114EU, Q4 HY12P03C2, SW1 SW_Push, U1 AP22615AWU-7, U10 TJA1042TK-3, U11 TJA1042TK-3, U12 XL1509-3.3, U13 USBLC6-2SC6, U3 10_0_QHHTZB6_3, U5 FM-B1921RGBA-SH, U6 TPS5450DDAR, U7 STM32H725ZGT6, U8 TJA1042TK-3, U9 TJA1042TK-3, Y1 25MHz X322525MOB4SI

Commit message: WIP: software verification pass in progress (reports, impedance, USB reroute, CPL rotation, DRC cleanup partial)
Co-authored-by: Copilot <223556219+Copilot@users.noreply.github.com>
Parts:
- moved R20 0.98 mm to (113.7, 44.0), turned to 90 degrees
- moved R21 0.58 mm to (114.8, 44.0), turned to -90 degrees
Routing:
- net USB_D-: track 3.30 -> 1.71 mm
- net GND: track 215.5 -> 214.2 mm, vias 96 -> 94
- net USB_R_D+: track 26.0 -> 24.9 mm, vias 2 -> 1
- net USB_PWR: track 31.1 -> 30.1 mm, vias 2 -> 0
- net USB_R_D-: track 24.2 -> 25.0 mm, vias 2 -> 1

Commit message: WIP: verification pass 1 complete (DRC 73 intentional, gerber connectivity 0 short/0 open, BOM fixes, hand-assembly edits, fab package regenerated)
Co-authored-by: Copilot <223556219+Copilot@users.noreply.github.com>
Routing:
- net GND: vias 94 -> 98
Changed lines of the file:
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@@
 		)
 		(pad_to_mask_clearance 0)
+		(solder_mask_min_width 0.1)
 		(allow_soldermask_bridges_in_footprints no)
 		(tenting
@@
 		(tags "capacitor")
 		(property "Reference" "C32"
-			(at 0 1.245391 0)
+			(at -1.3525 0 90)
 			(layer "F.SilkS")
 			(effects
@@
 		)
 		(fp_circle
-			(center -4.07 -1.905)
-			(end -3.97 -1.905)
+			(center -3.36 -2.69)
+			(end -3.26 -2.69)
 			(stroke
-				(width 0.2)
+				(width 0.15)
 				(type solid)
 			)
@@
 	)
 	(via
+		(at 126.695 55.245)
+		(size 0.6)
+		(drill 0.3)
+		(layers "F.Cu" "B.Cu")
+		(net "GND")
+	)
+	(via
 		(at 130.5 76)
 		(size 0.6)
@@
 	)
 	(via
+		(at 135.58 70.347)
+		(size 0.6)
+		(drill 0.3)
+		(layers "F.Cu" "B.Cu")
+		(net "GND")
+	)
+	(via
 		(at 106.62237 75.331277)
 		(size 0.7)
@@
 	)
 	(via
+		(at 127.5425 60.91)
+		(size 0.6)
+		(drill 0.3)
+		(layers "F.Cu" "B.Cu")
+		(net "GND")
+	)
+	(via
 		(at 108.25 65.862501)
 		(size 0.6)
@@
 	)
 	(via
+		(at 140.245 70.375)
+		(size 0.6)
+		(drill 0.3)
+		(layers "F.Cu" "B.Cu")
+		(net "GND")
+	)
+	(via
 		(at 125.018178 63.673367)
 		(size 0.6)
@@
 	)
 	(segment
+		(start 128.6 60.305)
+		(end 126.45 60.305)
+		(width 0.2)
+		(layer "In2.Cu")
+		(net "BUS1N_STB")
+	)
+	(segment
 		(start 121.6568 58.0382)
 		(end 119.5095 58.0382)
@@
 	)
 	(segment
-		(start 128.904 60.6092)
-		(end 123.9588 60.6092)
+		(start 126.146 60.609)
+		(end 123.959 60.609)
+		(width 0.2)
+		(layer "In2.Cu")
+		(net "BUS1N_STB")
+	)
+	(segment
+		(start 128.904 60.609)
+		(end 128.6 60.305)
+		(width 0.2)
+		(layer "In2.Cu")
+		(net "BUS1N_STB")
+	)
+	(segment
+		(start 126.45 60.305)
+		(end 126.146 60.609)
 		(width 0.2)
 		(layer "In2.Cu")
