File: hardware/hybrid-panda/HybridPanda.kicad_sch (KiCad schematic)
At the start: 119 parts, among them J1 SWD, P1 TYPE-C-31-M-04, Q1 DDTA143ECA-7-F P08, Q2 DDTA143ECA-7-F P08, Q3 PDTC114EU, Q4 HY12P03C2, SW1 SW_Push, U1 AP22615AWU-7, U10 TJA1042TK-3, U11 TJA1042TK-3, U12 XL1509-3.3, U13 USBLC6-2SC6, U3 10_0_QHHTZB6_3, U5 FM-B1921RGBA-SH, U6 TPS5450DDAR, U7 STM32H725ZGT6, U8 TJA1042TK-3, U9 TJA1042TK-3, Y1 25MHz X322525MOB4SI

Commit message: WIP: verification pass 1 complete (DRC 73 intentional, gerber connectivity 0 short/0 open, BOM fixes, hand-assembly edits, fab package regenerated)
Co-authored-by: Copilot <223556219+Copilot@users.noreply.github.com>
Parts:
- C23, C24: LCSC C1555 -> C1549
- C64: LCSC C23733 -> C12530; MPN CL05A225MP5NSNC -> CL05A225MQ5NSNC
